Commit message: Add range_node for the VL53L1X on the Pi, match the new launcher
New package pingpong_sensors with range_node: reads the VL53L1X over
the Pi I2C bus (narrowed to a 15 deg cone), median filter, publishes
/range/target. Started by the launch file on the real robot only.

The sensor is tilted 12 deg down from the barrel in the URDF, so its
cone still covers the target while the barrel is raised by the
ballistic elevation.

mock_hw_node simulates the new launcher (gear homing, cock to hold,
counted balls, RESET = refill) and the tilted 15 deg range cone.
The mission manager sends RESET to the launcher when the operator
resets with an empty magazine. Parameters updated for the OV5647
camera, the 7.9 m/s launcher and the 1-3.5 m range.

File: raspberry/src/pingpong_bringup/urdf/pingpong.urdf (robot description, URDF)
Before this commit: robot pingpong, 7 links, 6 joints
Joints:
- joint range_joint: origin xyz=0.12 0 0.04 rpy=0 0 0 -> xyz=0.12 0 0.04 rpy=0 0.21 0
